File: speed_cadence/hardware/Board1.kicad_sch (KiCad schematic)
At the start: 3 parts, among them IC1 AH1912-W-7, SW1 SW_Push, U1 STM32F042G6U6TR

Commit message: Major components added
Parts:
- added J1: DX07S016JA3R1500, DX07S016JA3R1500_USBC:CONN12_DX07S_JAE, symbol DX07S016JA3R1500_USBC:DX07S016JA3R1500
- added R1: 10K, Resistor_SMD:R_0603_1608Metric, symbol Device:R
- added U2: TS2940CW33_RPG, Package_TO_SOT_SMD:SOT-223-3_TabPin2, symbol TS2940CW33_RPG:TS2940CW33_RPG
- SW1: footprint (none) -> Button_Switch_SMD:SW_SPST_SKQG_WithStem
Connections:
- net VDD: now reaches IC1.1 (VDD)
- net VDD: now also U1.17 (VDD), R1.1
- net at IC1.2 (OUTPUT): now also U1.2 (PF0-OSC_IN)
- net GND: now reaches IC1.3 (GND)
- net GND: now also SW1.2, U1.16 (VSS)
- net at SW1.1: now also U1.4 (NRST), R1.2
Other:
- moved on the sheet: SW1

Commit message: Connected voltage regulator and fixed labels
Changed the VDD labels to the global labels that show voltage values. Added the capacitors for the voltage regulator
Parts:
- added C?: 22u, symbol Device:C_Polarized
- added C?: 0.47u, symbol Device:C_Polarized
Connections:
- net GND is gone; now on net +3V3: IC1.3 (GND), SW1.2, U1.16 (VSS)
- net +5V: now reaches U2.1 (INPUT)
- net +5V: now also IC1.1 (VDD), R1.1, C?.1
- net +3V3: now reaches U2.2 (GROUND_1)
- net +3V3: now also J1.1 (GND), J1.12 (GND), U1.17 (VDD), U2.4 (GROUND_2), C?.2, C?.2
- net at U2.3 (OUTPUT): now also C?.1
- removed net VDD: IC1.1 (VDD), R1.1, U1.17 (VDD)

Commit message: Added footprints for capacitors
Parts:
- C1, C2: renamed from C?; footprint (none) -> Capacitor_SMD:C_1206_3216Metric
Changed lines of the file:
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@@
 		(dnp no)
 		(fields_autoplaced yes)
-		(property "Reference" "C?"
+		(property "Reference" "C2"
 			(at 76.2 124.8409 0)
 			(effects
@@
 			)
 		)
-		(property "Footprint" ""
+		(property "Footprint" "Capacitor_SMD:C_1206_3216Metric"
 			(at 73.3552 130.81 0)
 			(effects
@@
 			(project "Board1"
 				(path "/10163266-8018-4064-a980-f3c4e9dfe9d4"
-					(reference "C?")
+					(reference "C2")
 					(unit 1)
 				)
@@
 		(dnp no)
 		(fields_autoplaced yes)
-		(property "Reference" "C?"
+		(property "Reference" "C1"
 			(at 58.42 117.2209 0)
 			(effects
@@
 			)
 		)
-		(property "Footprint" ""
+		(property "Footprint" "Capacitor_SMD:C_1206_3216Metric"
 			(at 55.5752 123.19 0)
 			(effects
@@
 			(project "Board1"
 				(path "/10163266-8018-4064-a980-f3c4e9dfe9d4"
-					(reference "C?")
-					(unit 1)
-				)
+					(reference "C1")
+					(unit 1)
+				)

Commit message: Updated voltage regulator output
Connections:
- net +3V3: now also C2.1, U2.3 (OUTPUT); no longer C1.2, C2.2, IC1.3 (GND), J1.1 (GND), J1.12 (GND), SW1.2, U1.16 (VSS), U2.2 (GROUND_1), U2.4 (GROUND_2)
- new net GND: C1.2, C2.2, IC1.3 (GND), J1.1 (GND), J1.12 (GND), SW1.2, U1.16 (VSS), U2.2 (GROUND_1), U2.4 (GROUND_2)
Changed lines of the file:
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@@
 	(paper "A4")
-	(junction
-		(at 115.57 109.22)
-		(diameter 0)
-		(color 0 0 0 0)
-	)
 	(junction
 		(at 54.61 109.22)
@@
 		(color 0 0 0 0)
 	)
+	(junction
+		(at 72.39 120.65)
+		(diameter 0)
+		(color 0 0 0 0)
+	)
 	(wire
 		(pts
@@
 	(wire
 		(pts
+			(xy 81.28 120.65) (xy 72.39 120.65)
+		)
+		(stroke
+			(width 0)
+			(type default)
+		)
+	)
+	(wire
+		(pts
 			(xy 149.86 93.98) (xy 149.86 99.06)
 		)
@@
 	(wire
 		(pts
-			(xy 115.57 109.22) (xy 124.46 109.22)
-		)
-		(stroke
-			(width 0)
-			(type default)
-		)
-	)
-	(wire
-		(pts
 			(xy 203.2 124.46) (xy 196.85 124.46)
 		)
@@
 	(wire
 		(pts
-			(xy 72.39 114.3) (xy 72.39 123.19)
+			(xy 72.39 114.3) (xy 72.39 120.65)
 		)
 		(stroke
@@
 		(pts
 			(xy 190.5 74.93) (xy 180.34 64.77)
+		)
+		(stroke
+			(width 0)
+			(type default)
+		)
+	)
+	(wire
+		(pts
+			(xy 72.39 120.65) (xy 72.39 123.19)
 		)
 		(stroke
@@
 	)
 	(symbol
+		(lib_id "power:+3V3")
+		(at 81.28 120.65 270)
+		(unit 1)
+		(exclude_from_sim no)
+		(in_bom yes)
+		(on_board yes)
+		(dnp no)
+		(fields_autoplaced yes)
+		(property "Reference" "#PWR013"
+			(at 77.47 120.65 0)
+			(effects
+				(font
+					(size 1.27 1.27)
+				)
+				(hide yes)
+			)
+		)
+		(property "Value" "+3V3"
+			(at 85.09 120.6499 90)
+			(effects
+				(font
+					(size 1.27 1.27)
+				)
+				(justify left)
+			)
+		)
+		(property "Footprint" ""
+			(at 81.28 120.65 0)
+			(effects
+				(font
+					(size 1.27 1.27)
+				)
+				(hide yes)
+			)
+		)
+		(property "Datasheet" ""
+			(at 81.28 120.65 0)
+			(effects
+				(font
+					(size 1.27 1.27)
+				)
+				(hide yes)
+			)
+		)
+		(property "Description" "Power symbol creates a global label with name \"+3V3\""
+			(at 81.28 120.65 0)
+			(effects
+				(font
+					(size 1.27 1.27)
+				)
+				(hide yes)
+			)
+		)
+		(pin "1"
+		)
+		(instances
+			(project "Board1"
+				(path "/10163266-8018-4064-a980-f3c4e9dfe9d4"
+					(reference "#PWR013")
+					(unit 1)
+				)
+			)
+		)
+	)
+	(symbol
 		(lib_id "Device:C_Polarized")
 		(at 72.39 127 0)
@@
 					(unit 1)
 				)
-			)
-		)
-	)
-	(symbol
-		(lib_id "power:+3V3")
-		(at 124.46 109.22 270)
-		(unit 1)
-		(exclude_from_sim no)
-		(in_bom yes)
-		(on_board yes)
-		(dnp no)
-		(fields_autoplaced yes)
-		(property "Reference" "#PWR013"
-			(at 120.65 109.22 0)
-			(effects
-				(font
-					(size 1.27 1.27)
-				)
-				(hide yes)
-			)
-		)
-		(property "Value" "+3V3"
-			(at 128.27 109.2199 90)
-			(effects
-				(font
-					(size 1.27 1.27)
-				)
-				(justify left)
-			)
-		)
-		(property "Footprint" ""
-			(at 124.46 109.22 0)
-			(effects
-				(font
-					(size 1.27 1.27)
-				)
-				(hide yes)
-			)
-		)
-		(property "Datasheet" ""
-			(at 124.46 109.22 0)
-			(effects
-				(font
-					(size 1.27 1.27)
-				)
-				(hide yes)
-			)
-		)
-		(property "Description" "Power symbol creates a global label with name \"+3V3\""
-			(at 124.46 109.22 0)
-			(effects
-				(font
-					(size 1.27 1.27)
-				)
-				(hide yes)
-			)
-		)
-		(pin "1"
-		)
-		(instances
-			(project "Board1"
-				(path "/10163266-8018-4064-a980-f3c4e9dfe9d4"
-					(reference "#PWR013")
-					(unit 1)
-				)

Commit message: Connected USB-C to microcontroller
Parts:
- added R? (x2): 5.1k, Resistor_SMD:R_0603_1608Metric, symbol Device:R
Connections:
- net +5V: now also J1.11 (VBUS), J1.2 (VBUS)
- net GND: now also R?.2, R?.2
- net at U1.19 (PA9/PA11): now also J1.5 (D-), J1.8 (D-)
- net at U1.20 (PA10/PA12): now also J1.6 (D+), J1.7 (D+)
- net at J1.3 (CC1): now also R?.1
- net at J1.9 (CC2): now also R?.1
- no-connect marks 0 -> 24
Other:
- moved on the sheet: J1

Commit message: Resistors named
Parts:
- gave numbers to parts that had none: 2
Changed lines of the file:
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@@
 		(dnp no)
 		(fields_autoplaced yes)
-		(property "Reference" "R?"
+		(property "Reference" "R2"
 			(at 31.75 53.3399 0)
 			(effects
@@
 			(project "Board1"
 				(path "/10163266-8018-4064-a980-f3c4e9dfe9d4"
-					(reference "R?")
+					(reference "R2")
 					(unit 1)
 				)
@@
 		(dnp no)
 		(fields_autoplaced yes)
-		(property "Reference" "R?"
+		(property "Reference" "R3"
 			(at 31.75 73.6599 0)
 			(effects
@@
 			(project "Board1"
 				(path "/10163266-8018-4064-a980-f3c4e9dfe9d4"
-					(reference "R?")
+					(reference "R3")
 					(unit 1)
 				)
