File: speed_cadence/hardware/Board1.kicad_sch (KiCad schematic)
At the start: 17 parts, among them IC1 AH1912-W-7, J1 DX07S016JA3R1500, J2 Conn_01x04_Pin, J3 Conn_ST_STDC14, SW1 SW_Push, U1 STM32F042G6U6TR, U2 TS2940CW33_RPG, U4 TJA1051T-3

Commit message: Updated differential pair routing
CANH is now CAN+
CANL is now CAN- for KiCAD to recognize the differential pair.
Connections:
- net CAN_H renamed CAN+
- net CAN_L renamed CAN-
Changed lines of the file:
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@@
 		)
 	)
-	(global_label "CAN_H"
+	(global_label "CAN+"
 		(shape input)
 		(at 113.03 168.91 0)
@@
 		)
 		(property "Intersheetrefs" "${INTERSHEET_REFS}"
-			(at 122.0024 168.91 0)
+			(at 121.2767 168.91 0)
 			(effects
 				(font
@@
 		)
 	)
-	(global_label "CAN_L"
+	(global_label "CAN-"
 		(shape input)
 		(at 52.07 134.62 0)
@@
 		)
 		(property "Intersheetrefs" "${INTERSHEET_REFS}"
-			(at 60.74 134.62 0)
+			(at 60.3167 134.62 0)
 			(effects
 				(font
@@
 		)
 	)
-	(global_label "CAN_H"
+	(global_label "CAN+"
 		(shape input)
 		(at 52.07 127 0)
@@
 		)
 		(property "Intersheetrefs" "${INTERSHEET_REFS}"
-			(at 61.0424 127 0)
+			(at 60.3167 127 0)
 			(effects
 				(font
@@
 		)
 	)
-	(global_label "CAN_L"
+	(global_label "CAN-"
 		(shape input)
 		(at 113.03 172.72 0)
@@
 		)
 		(property "Intersheetrefs" "${INTERSHEET_REFS}"
-			(at 121.7 172.72 0)
+			(at 121.2767 172.72 0)
 			(effects
 				(font
