File: speed_cadence/hardware/Board1.kicad_pcb (KiCad board)
At the start: 2 copper layers, 39.4 x 46.4 mm, 15 parts, among them IC1 AH1912-W-7, J1 DX07S016JA3R1500, J2 Conn_01x04_Pin, SW1 SW_Push, U1 STM32F042G6U6TR, U2 TS2940CW33_RPG

Commit message: Replaced things
Parts:
- moved H4 37.2 mm to (96.4, 93.4)
- moved H1 36.8 mm to (96.4, 57.2)
- moved C1 14.4 mm to (88.2, 65.2), turned to -90 degrees
- moved C2 14.0 mm to (88.2, 70.2), turned to 90 degrees
- moved SW1 13.9 mm to (86.4, 57.0), turned to 180 degrees
- moved U2 13.1 mm to (94.3, 67.6)
- moved R1 11.8 mm to (80.2, 58.8), turned to 0 degrees
- moved J2 8.99 mm to (74.2, 77.0), turned to 0 degrees
- moved J1 6.55 mm to (75.5, 67.6), turned to -90 degrees
- moved R2 6.21 mm to (81.4, 65.1), turned to 90 degrees
- moved U1 5.63 mm to (92.6, 79.0)
- moved IC1 4.40 mm to (84.6, 93.6)
- moved R3 2.05 mm to (81.4, 69.5)
Routing:
- net +5V: track 65.1 -> 0.00 mm, vias 1 -> 0
- net CAN_RX: track 48.5 -> 0.00 mm, vias 4 -> 0
- net CAN_TX: track 44.2 -> 0.00 mm, vias 2 -> 0
- net Net-(U1A-NRST): track 27.8 -> 0.00 mm
- net Net-(IC1-OUTPUT): track 25.3 -> 0.00 mm, vias 1 -> 0
- net +3V3: track 18.4 -> 0.00 mm, vias 2 -> 0
- net GND: track 18.2 -> 0.00 mm, vias 11 -> 0
- net Net-(J1-CC1): track 7.40 -> 0.00 mm, vias 2 -> 0
- net Net-(J1-CC2): track 6.43 -> 0.00 mm, vias 2 -> 0
- removed copper zone on B.Cu, net GND
Other:
- board size 39.4 x 46.4 mm -> 32.8 x 46.4 mm

Commit message: New routing
Routing:
- net +5V: track 0.00 -> 56.1 mm
- net CAN_RX: track 0.00 -> 43.8 mm, vias 0 -> 2
- net CAN_TX: track 0.00 -> 39.6 mm, vias 0 -> 2
- net Net-(U1A-NRST): track 0.00 -> 33.0 mm
- net Net-(IC1-OUTPUT): track 0.00 -> 23.3 mm, vias 0 -> 1
- net +3V3: track 0.00 -> 12.5 mm
- net Net-(J1-CC2): track 0.00 -> 2.69 mm
- net Net-(J1-CC1): track 0.00 -> 2.66 mm

Commit message: added ground pour
Routing:
- added copper zone on F.Cu, net GND
Changed lines of the file:
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@@
 	)
 	(gr_text "SPEED MEASUREMENT - TYPHOON\nEVELYN KOSZTA and EUN GU KANG"
-		(at 85 88.4 -0)
+		(at 85 88.4 0)
 		(layer "F.SilkS")
 		(effects
 			(font
 				(size 0.8 0.8)
-				(thickness 0.07)
-				(bold yes)
+				(thickness 0.08)
 			)
 			(justify bottom)
@@
 		(net 33)
 	)
+	(zone
+		(net 2)
+		(net_name "GND")
+		(layer "F.Cu")
+		(hatch edge 0.5)
+		(connect_pads
+			(clearance 0.5)
+		)
+		(min_thickness 0.25)
+		(filled_areas_thickness no)
+		(fill yes
+			(thermal_gap 0.5)
+			(thermal_bridge_width 0.5)
+		)
+		(polygon
+			(pts
+				(xy 71 52) (xy 99.4 52) (xy 101.2 53.8) (xy 101.2 94.8) (xy 98.4 97.6) (xy 71.6 97.6) (xy 69.2 95.2)
+				(xy 69.2 53.8)
+			)
+		)
+	)
 )

Commit message: updated tracks
Routing:
- net GND: track 0.00 -> 2.71 mm
Changed lines of the file:
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@@
 			(at 0 -3.75 0)
 			(layer "F.SilkS")
+			(hide yes)
 			(effects
 				(font
@@
 			(at 0 -3.75 0)
 			(layer "F.SilkS")
+			(hide yes)
 			(effects
 				(font
@@
 			(at 0 -3.75 0)
 			(layer "F.SilkS")
+			(hide yes)
 			(effects
 				(font
@@
 			(at 0 -3.75 0)
 			(layer "F.SilkS")
+			(hide yes)
 			(effects
 				(font
@@
 	)
 	(segment
+		(start 79.005691 64.239732)
+		(end 81.365689 64.239732)
+		(width 0.2)
+		(layer "F.Cu")
+		(net 2)
+	)
+	(segment
+		(start 78.760689 64.484734)
+		(end 79.005691 64.239732)
+		(width 0.2)
+		(layer "F.Cu")
+		(net 2)
+	)
+	(segment
