File: environmentals/hardware/env_sens_Kicad/env_sens.kicad_pcb (KiCad board)
At the start: 2 copper layers, 40 parts, among them J1 CO2_Conn, J2 BATTERY, J3 USB_C_Receptacle_USB2.0_14P, J4 CAN_BUS, SW1 RESET, SW2 BOOT, U1 HDC1080, U2 TCAN1043xDxQ1, U3 ESP32-S3-WROOM-1, U6 TPD1E05U06DYA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

Commit message: Finished environmental board layout
Parts:
- C11: footprint Capacitor_SMD:C_0805_2012Metric_Pad1.18x1.45mm_HandSolder -> Capacitor_SMD:C_0603_1608Metric_Pad1.08x0.95mm_HandSolder
- J3: footprint Connector_USB:USB_C_Receptacle_Amphenol_12401548E4-2A_CircularHoles -> Connector_USB:USB_C_Receptacle_Amphenol_12401610E4-2A
- R5, R6: footprint Resistor_SMD:R_0805_2012Metric_Pad1.20x1.40mm_HandSolder -> Resistor_SMD:R_0603_1608Metric_Pad0.98x0.95mm_HandSolder
- moved D1 140.7 mm to (36.0, 43.5), turned to 90 degrees
- moved J1 119.8 mm to (44.0, 28.2), turned to -90 degrees
- moved H2 117.6 mm to (39.8, 21.8)
- moved R7 111.2 mm to (36.0, 39.5), turned to -90 degrees
- moved H3 109.7 mm to (39.8, 71.8)
- moved C5 109.3 mm to (49.8, 22.9), turned to -90 degrees
- moved R1 108.2 mm to (47.8, 22.8), turned to -90 degrees
- moved U6 107.3 mm to (61.8, 68.8), turned to 90 degrees
- moved U7 103.9 mm to (68.5, 64.5)
- moved U1 102.1 mm to (90.8, 30.1)
- moved SW1 100.2 mm to (52.2, 42.0), turned to -90 degrees
- moved C4 97.0 mm to (39.5, 47.5), turned to 180 degrees
- moved SW2 95.8 mm to (59.0, 48.5), turned to 90 degrees
- moved U2 92.1 mm to (79.2, 53.2), turned to -90 degrees
- moved C3 91.9 mm to (42.0, 49.8), turned to 180 degrees
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Connections:
- net /USB_D+ renamed /USB_D_P
- net /USB_D- renamed /USB_D_N
- J4 pad 1: /CANH -> /CANL
- J4 pad 2: /CANL -> /CANH
- R3 pad 2: /I2C1_SCL -> /I2C1_SDA
- U1 pad 1: /I2C1_SCL -> /I2C1_SDA
- U3 pad 10: unconnected-(U3-IO17-Pad10) -> /CO2_PWM
- U3 pad 12: /CAN_STBn -> unconnected-(U3-IO8-Pad12)
- U3 pad 15: /I2C1_SCL -> unconnected-(U3-IO3-Pad15)
- U3 pad 17: /CO2_PWM -> unconnected-(U3-IO9-Pad17)
- U3 pad 29: unconnected-(U3-IO36-Pad29) -> /CAN_FAULTn
- U3 pad 30: unconnected-(U3-IO37-Pad30) -> /CAN_EN
- U3 pad 31: unconnected-(U3-IO38-Pad31) -> /CAN_RX
- U3 pad 32: unconnected-(U3-IO39-Pad32) -> /CAN_TX
- U3 pad 33: unconnected-(U3-IO40-Pad33) -> /CAN_STBn
- U3 pad 34: unconnected-(U3-IO41-Pad34) -> /I2C1_SDA
- U3 pad 35: unconnected-(U3-IO42-Pad35) -> /I2C1_SCL
- U3 pad 38: /I2C1_SCL -> unconnected-(U3-IO2-Pad38)
- U3 pad 4: /CAN_RX -> unconnected-(U3-IO4-Pad4)
- U3 pad 5: /CAN_TX -> unconnected-(U3-IO5-Pad5)
- U3 pad 6: /CAN_EN -> unconnected-(U3-IO6-Pad6)
- U3 pad 7: /CAN_FAULTn -> unconnected-(U3-IO7-Pad7)
Routing:
- net +3V3: track 0.00 -> 114.8 mm, vias 0 -> 6
- net +5V: track 0.00 -> 104.2 mm, vias 0 -> 2
- net GND: track 0.00 -> 61.8 mm, vias 0 -> 22
- net /USB_D_N: track 0.00 -> 44.4 mm, vias 0 -> 4
- net /USB_D_P: track 0.00 -> 41.7 mm, vias 0 -> 3
- net /CAN_STBn: track 0.00 -> 36.3 mm
- net Net-(U3-EN): track 0.00 -> 30.6 mm, vias 0 -> 2
- net /CAN_TX: track 0.00 -> 28.7 mm
- net /CAN_FAULTn: track 0.00 -> 26.2 mm
- net Net-(J3-SHIELD): track 0.00 -> 26.1 mm, vias 0 -> 2
- net /CAN_RX: track 0.00 -> 25.4 mm
- net /I2C1_SCL: track 0.00 -> 24.3 mm
- net /CAN_EN: track 0.00 -> 23.0 mm
- net /I2C1_SDA: track 0.00 -> 21.0 mm
- net Net-(U3-IO0): track 0.00 -> 17.1 mm
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- added copper zone on B.Cu, net GND
Other:
- board outline added: 60 x 60 mm
- board text added: "DO NOT CONNECT USB AND BATTERY AT THE SAME TIME"
