File: environmentals/hardware/env_sens_Kicad/env_sens.kicad_sch (KiCad schematic)
At the start: 40 parts, among them J1 CO2_Conn, J2 BATTERY, J3 USB_C_Receptacle_USB2.0_14P, J4 CAN_BUS, SW1 RESET, SW2 BOOT, U1 HDC1080, U2 TCAN1043xDxQ1, U3 ESP32-S3-WROOM-1, U6 TPD1E05U06DYA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

Commit message: Finished environmental board layout
Parts:
- C11: footprint Capacitor_SMD:C_0805_2012Metric_Pad1.18x1.45mm_HandSolder -> Capacitor_SMD:C_0603_1608Metric_Pad1.08x0.95mm_HandSolder
- J3: footprint Connector_USB:USB_C_Receptacle_Amphenol_12401548E4-2A_CircularHoles -> Connector_USB:USB_C_Receptacle_Amphenol_12401610E4-2A
- R5, R6: footprint Resistor_SMD:R_0805_2012Metric_Pad1.20x1.40mm_HandSolder -> Resistor_SMD:R_0603_1608Metric_Pad0.98x0.95mm_HandSolder
Connections:
- net CANH: now also J4.2 (Pin_2); no longer J4.1 (Pin_1)
- net CANL: now also J4.1 (Pin_1); no longer J4.2 (Pin_2)
- net CAN_EN: now also U3.30 (IO37); no longer U3.6 (IO6)
- net CAN_FAULTn: now also U3.29 (IO36); no longer U3.7 (IO7)
- net CAN_RX: now also U3.31 (IO38); no longer U3.4 (IO4)
- net CAN_STBn: now also U3.33 (IO40); no longer U3.12 (IO8)
- net CAN_TX: now also U3.32 (IO39); no longer U3.5 (IO5)
- net CO2_PWM: now also U3.10 (IO17); no longer U3.17 (IO9)
- net I2C1_SCL: now also U3.35 (IO42); no longer R3.2, U1.1 (SDA), U3.15 (IO3), U3.38 (IO2)
- net I2C1_SDA: now reaches U3.34 (IO41)
- net I2C1_SDA: now also R3.2, U1.1 (SDA)
- net USB_D+ renamed USB_D_P
- net USB_D- renamed USB_D_N
Other:
- moved on the sheet: R3
