File: motherboard/hardware/Typhoon Motherboard KiCad/Typhoon Motherboard KiCad.kicad_sch (KiCad schematic)
At the start: 10 parts, among them J1 Conn_01x04_Pin, P1 USB_C_Plug_USB2.0, U1 ESP32-S3-WROOM-1, U2 AZ1117-3.3

Commit message: added footprint for CAN transceiver
Parts:
- U3: footprint (none) -> Package_SO:SO-8_3.9x4.9mm_P1.27mm
Changed lines of the file:
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@@
 			)
 		)
-		(property "Footprint" ""
+		(property "Footprint" "Package_SO:SO-8_3.9x4.9mm_P1.27mm"
 			(at 198.12 83.82 0)
 			(effects
