File: power/hardware/powermeter/powermeter.kicad_sch (KiCad schematic)
At the start: 16 parts, among them J1 Conn_01x02_Socket, J2 Conn_01x04_Pin, P1 USB_C_Plug_USB2.0, U2 ESP32-S3-WROOM-1, U3 AZ1117-3.3

Commit message: added pcb
Parts:
- removed C4: 100n, symbol Device:C
- added C12: 10n, Capacitor_SMD:C_0603_1608Metric, symbol Device:C
- added C13: 1u, Capacitor_SMD:C_0603_1608Metric, symbol Device:C
- added C8: 100n, Capacitor_SMD:C_0603_1608Metric, symbol Device:C
- added J3: Conn_01x02_Socket, Connector_AMASS:AMASS_XT30U-M_1x02_P5.0mm_Vertical, symbol Connector:Conn_01x02_Pin
- added U1: ~, Package_SO:SO-8_3.9x4.9mm_P1.27mm, symbol Interface_CAN_LIN:TJA1051
- ADS131M03: footprint (none) -> 0_stuff:ads
- C1, C2, C5: footprint (none) -> Capacitor_SMD:C_0603_1608Metric
- C3: value 100n -> 1u; footprint (none) -> Capacitor_SMD:C_0603_1608Metric
- J1: footprint (none) -> Connector_PinHeader_2.00mm:PinHeader_1x02_P2.00mm_Vertical; symbol Connector:Conn_01x02_Socket -> Connector:Conn_01x02_Pin
- MPU6000: footprint (none) -> 0_stuff:QFN24_4X4X0P9_IVS
- P1: footprint (none) -> Connector_USB:USB_C_Receptacle_HRO_TYPE-C-31-M-12
- R1, R2: footprint (none) -> Resistor_SMD:R_0603_1608Metric
Connections:
- net +3V3: now also C12.2, C13.2, C8.2, J3.2 (Pin_2), U1.3 (V_{CC})
- net CANH: now also U1.7 (CANH); no longer U2.8 (IO15)
- net CANL: now also U1.6 (CANL); no longer U2.9 (IO16)
- net CLK_{ADC}: now also U2.16 (IO46); no longer U2.34 (IO41)
- net CS_{ADC}: now also U2.18 (IO10); no longer U2.6 (IO6)
- net CS_{gyro}: now also U2.26 (IO45); no longer U2.4 (IO4)
- net DRDY_{ADC}: now also U2.17 (IO9); no longer U2.12 (IO8)
- net GND: now also C12.1, C13.1, C8.1, J3.1 (Pin_1), U1.2 (GND), U1.8 (S)
- net INT_{gyro}: now also U2.25 (IO48); no longer U2.5 (IO5)
- net MOSI: now also U2.20 (IO12); no longer U2.19 (IO11)
- net SCLK: now also U2.22 (IO14); no longer U2.20 (IO12)
- net SYNC_{ADC}: now also U2.19 (IO11); no longer U2.7 (IO7)
- net ADS-: now reaches ADS131M03.2 (AIN0N), J1.1 (Pin_1)
- net ADS+: now reaches ADS131M03.1 (AIN0P), J1.2 (Pin_2)
- net TX: now reaches U2.11 (IO18)
- net TX: now also U1.1 (TXD)
- net USB_{D+} renamed USB_{D}+
- net USB_{D-} renamed USB_{D}-
- new net RX: U1.4 (RXD), U2.12 (IO8)
Other:
- moved on the sheet: C1, C2, C3, C6, C7, J2, MPU6000, P1, R1, R2, U3

Commit message: updated pcb
Parts:
- removed J1: Conn_01x02_Socket, Connector_PinHeader_2.00mm:PinHeader_1x02_P2.00mm_Vertical, symbol Connector:Conn_01x02_Pin
- added J4: Conn_01x04_Pin, Connector_PinHeader_2.00mm:PinHeader_1x04_P2.00mm_Vertical, symbol Connector:Conn_01x04_Pin
- renumbered C5 to C4, C6 to C5, C7 to C6, C8 to C7, C12 to C8, C13 to C9
Connections:
- net +3V3: now also J4.1 (Pin_1)
- net ADS+: now also J4.3 (Pin_3)
- net ADS-: now also J4.4 (Pin_4)
- net GND: now also J4.2 (Pin_2)
Changed lines of the file:
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@@
 	(wire
 		(pts
+			(xy 33.02 71.12) (xy 25.4 71.12)
+		)
+		(stroke
+			(width 0)
+			(type default)
+		)
+	)
+	(wire
+		(pts
 			(xy 140.97 81.28) (xy 144.78 81.28)
 		)
@@
 	(wire
 		(pts
+			(xy 33.02 73.66) (xy 25.4 73.66)
+		)
+		(stroke
+			(width 0)
+			(type default)
+		)
+	)
+	(wire
+		(pts
 			(xy 144.78 138.43) (xy 140.97 138.43)
 		)
@@
 	(text "wheatstone bridge\nvoltage measurement\ngoes here"
 		(exclude_from_sim no)
-		(at 27.432 47.752 0)
+		(at 22.606 61.468 0)
 		(effects
 			(font
@@
 		)
 	)
+	(label "ADS-"
+		(at 25.4 78.74 0)
+		(fields_autoplaced yes)
+		(effects
+			(font
+				(size 1.27 1.27)
+			)
+			(justify left bottom)
+		)
+	)
 	(label "DRDY_{ADC}"
 		(at 72.39 69.85 0)
@@
 		)
 	)
-	(label "ADS+"
-		(at 24.13 59.69 0)
-		(fields_autoplaced yes)
-		(effects
-			(font
-				(size 1.27 1.27)
-			)
-			(justify left bottom)
-		)
-	)
 	(label "USB_{D}+"
 		(at 107.95 68.58 180)
@@
 		)
 	)
+	(label "ADS+"
+		(at 25.4 76.2 0)
+		(fields_autoplaced yes)
+		(effects
+			(font
+				(size 1.27 1.27)
+			)
+			(justify left bottom)
+		)
+	)
 	(label "INT_{gyro}"
 		(at 200.66 68.58 0)
@@
 		)
 	)
-	(label "ADS-"
-		(at 24.13 62.23 0)
-		(fields_autoplaced yes)
-		(effects
-			(font
-				(size 1.27 1.27)
-			)
-			(justify left bottom)
-		)
-	)
 	(label "MISO"
 		(at 144.78 93.98 0)
@@
 	)
 	(symbol
+		(lib_id "power:GND")
+		(at 33.02 73.66 0)
+		(unit 1)
+		(exclude_from_sim no)
+		(in_bom yes)
+		(on_board yes)
+		(dnp no)
+		(fields_autoplaced yes)
+		(property "Reference" "#PWR027"
+			(at 33.02 80.01 0)
+			(effects
+				(font
+					(size 1.27 1.27)
+				)
+				(hide yes)
+			)
+		)
+		(property "Value" "GND"
+			(at 33.02 78.74 0)
+			(effects
+				(font
+					(size 1.27 1.27)
+				)
+			)
+		)
+		(property "Footprint" ""
+			(at 33.02 73.66 0)
+			(effects
+				(font
+					(size 1.27 1.27)
+				)
+				(hide yes)
+			)
+		)
+		(property "Datasheet" ""
+			(at 33.02 73.66 0)
+			(effects
+				(font
+					(size 1.27 1.27)
+				)
+				(hide yes)
+			)
+		)
+		(property "Description" "Power symbol creates a global label with name \"GND\" , ground"
+			(at 33.02 73.66 0)
+			(effects
+				(font
+					(size 1.27 1.27)
+				)
+				(hide yes)
+			)
+		)
+		(pin "1"
+		)
+		(instances
+			(project "powermeter"
+				(path "/ff8c320c-6506-4f89-8e94-bef2c667bd19"
+					(reference "#PWR027")
+					(unit 1)
+				)
+			)
+		)
+	)
+	(symbol
 		(lib_id "power:+3V3")
 		(at 107.95 135.89 0)
@@
 	)
 	(symbol
-		(lib_id "Connector:Conn_01x02_Pin")
-		(at 19.05 62.23 0)
-		(mirror x)
-		(unit 1)
-		(exclude_from_sim no)
-		(in_bom yes)
-		(on_board yes)
-		(dnp no)
-		(property "Reference" "J1"
-			(at 21.844 52.324 0)
-			(effects
-				(font
-					(size 1.27 1.27)
-				)
-			)
-		)
-		(property "Value" "Conn_01x02_Socket"
-			(at 22.606 54.864 0)
-			(effects
-				(font
-					(size 1.27 1.27)
-				)
-			)
-		)
-		(property "Footprint" "Connector_PinHeader_2.00mm:PinHeader_1x02_P2.00mm_Vertical"
-			(at 19.05 62.23 0)
-			(effects
-				(font
-					(size 1.27 1.27)
-				)
-				(hide yes)
-			)
-		)
-		(property "Datasheet" "~"
-			(at 19.05 62.23 0)
-			(effects
-				(font
-					(size 1.27 1.27)
-				)
-				(hide yes)
-			)
-		)
-		(property "Description" "Generic connector, single row, 01x02, script generated"
-			(at 19.05 62.23 0)
-			(effects
-				(font
-					(size 1.27 1.27)
-				)
-				(hide yes)
-			)
-		)
-		(pin "1"
-		)
-		(pin "2"
-		)
-		(instances
-			(project "powermeter"
-				(path "/ff8c320c-6506-4f89-8e94-bef2c667bd19"
-					(reference "J1")
-					(unit 1)
-				)
-			)
-		)
-	)
-	(symbol
 		(lib_id "power:GND")
 		(at 139.7 43.18 0)
@@
 		(on_board yes)
 		(dnp no)
-		(property "Reference" "C5"
+		(property "Reference" "C4"
 			(at 61.976 78.994 0)
 			(effects
@@
 			(project "powermeter"
 				(path "/ff8c320c-6506-4f89-8e94-bef2c667bd19"
-					(reference "C5")
+					(reference "C4")
 					(unit 1)
 				)
@@
 	)
 	(symbol
+		(lib_id "Connector:Conn_01x04_Pin")
+		(at 20.32 73.66 0)
+		(unit 1)
+		(exclude_from_sim no)
+		(in_bom yes)
+		(on_board yes)
+		(dnp no)
+		(fields_autoplaced yes)
+		(property "Reference" "J4"
+			(at 20.955 66.04 0)
+			(effects
+				(font
+					(size 1.27 1.27)
+				)
+			)
+		)
+		(property "Value" "Conn_01x04_Pin"
+			(at 20.955 68.58 0)
+			(effects
+				(font
+					(size 1.27 1.27)
+				)
+			)
+		)
+		(property "Footprint" "Connector_PinHeader_2.00mm:PinHeader_1x04_P2.00mm_Vertical"
+			(at 20.32 73.66 0)
+			(effects
+				(font
+					(size 1.27 1.27)
+				)
+				(hide yes)
+			)
+		)
+		(property "Datasheet" "~"
+			(at 20.32 73.66 0)
+			(effects
+				(font
+					(size 1.27 1.27)
+				)
+				(hide yes)
+			)
+		)
+		(property "Description" "Generic connector, single row, 01x04, script generated"
+			(at 20.32 73.66 0)
+			(effects
+				(font
+					(size 1.27 1.27)
+				)
+				(hide yes)
+			)
+		)
+		(pin "4"
+		)
+		(pin "2"
+		)
+		(pin "1"
+		)
+		(pin "3"
+		)
+		(instances
+			(project "powermeter"
+				(path "/ff8c320c-6506-4f89-8e94-bef2c667bd19"
+					(reference "J4")
+					(unit 1)
+				)
+			)
+		)
+	)
+	(symbol
 		(lib_id "power:GND")
 		(at 210.82 57.15 0)
@@
 		(on_board yes)
 		(dnp no)
-		(property "Reference" "C7"
+		(property "Reference" "C6"
 			(at 146.05 144.78 0)
 			(effects
@@
 			(project "powermeter"
 				(path "/ff8c320c-6506-4f89-8e94-bef2c667bd19"
-					(reference "C7")
+					(reference "C6")
 					(unit 1)
 				)
@@
 	(symbol
 		(lib_id "power:+3V3")
+		(at 33.02 71.12 0)
+		(unit 1)
+		(exclude_from_sim no)
+		(in_bom yes)
+		(on_board yes)
+		(dnp no)
+		(property "Reference" "#PWR026"
+			(at 33.02 74.93 0)
+			(effects
+				(font
+					(size 1.27 1.27)
+				)
+				(hide yes)
+			)
+		)
+		(property "Value" "+3V3"
+			(at 32.766 67.31 0)
+			(effects
+				(font
+					(size 1.27 1.27)
+				)
+			)
+		)
+		(property "Footprint" ""
+			(at 33.02 71.12 0)
+			(effects
+				(font
+					(size 1.27 1.27)
+				)
+				(hide yes)
+			)
+		)
+		(property "Datasheet" ""
+			(at 33.02 71.12 0)
+			(effects
+				(font
+					(size 1.27 1.27)
+				)
+				(hide yes)
+			)
+		)
+		(property "Description" "Power symbol creates a global label with name \"+3V3\""
+			(at 33.02 71.12 0)
+			(effects
+				(font
+					(size 1.27 1.27)
+				)
+				(hide yes)
+			)
+		)
+		(pin "1"
+		)
+		(instances
+			(project "powermeter"
+				(path "/ff8c320c-6506-4f89-8e94-bef2c667bd19"
+					(reference "#PWR026")
+					(unit 1)
+				)
+			)
+		)
+	)
+	(symbol
+		(lib_id "power:+3V3")
 		(at 182.88 50.8 0)
 		(unit 1)
@@
 		(on_board yes)
 		(dnp no)
-		(property "Reference" "C6"
+		(property "Reference" "C5"
 			(at 118.11 144.78 0)
 			(effects
@@
 			(project "powermeter"
 				(path "/ff8c320c-6506-4f89-8e94-bef2c667bd19"
-					(reference "C6")
+					(reference "C5")
 					(unit 1)
 				)
@@
 		(on_board yes)
 		(dnp no)
-		(property "Reference" "C8"
+		(property "Reference" "C7"
 			(at 130.556 38.608 0)
 			(effects
@@
 			(project "powermeter"
 				(path "/ff8c320c-6506-4f89-8e94-bef2c667bd19"
-					(reference "C8")
+					(reference "C7")
 					(unit 1)
 				)
@@
 		(on_board yes)
 		(dnp no)
-		(property "Reference" "C12"
+		(property "Reference" "C8"
 			(at 140.716 38.608 0)
 			(effects
@@
 			(project "powermeter"
 				(path "/ff8c320c-6506-4f89-8e94-bef2c667bd19"
-					(reference "C12")
+					(reference "C8")
 					(unit 1)
 				)
@@
 		(on_board yes)
 		(dnp no)
-		(property "Reference" "C13"
+		(property "Reference" "C9"
 			(at 149.86 38.354 0)
 			(effects
@@
 			(project "powermeter"
 				(path "/ff8c320c-6506-4f89-8e94-bef2c667bd19"
-					(reference "C13")
+					(reference "C9")
 					(unit 1)
 				)
